File: KiCad/pcb-hat-thermo/pcb-hat-thermo.kicad_pcb (KiCad board)
At the start: 2 copper layers, 65.5 x 30.5 mm, 7 parts, among them J1 Screw_Terminal_01x03, J2 Screw_Terminal_01x03, J3 Screw_Terminal_01x03, J4 Screw_Terminal_01x03, J5 Screw_Terminal_01x03, J6 Raspberry_Pi_2_3

Commit message: Version 1.0
Parts:
- J1, J2, J3, J4, J5: footprint TerminalBlock_4Ucon:TerminalBlock_4Ucon_1x03_P3.50mm_Horizontal -> Connector_Phoenix_MC:PhoenixContact_MC_1,5_3-G-3.5_1x03_P3.50mm_Horizontal
- J6: footprint pcb-hat-lib:Raspberry_Pi_Zero_Custom -> pcb-hat-lib:Raspberry_Pi_Zero_Custom_with_Header
- moved J1 3.94 mm to (98.5, 99.0)
- moved J2 3.91 mm to (111.4, 102.3)
- moved J3 3.91 mm to (126.3, 102.3)
- moved J4 3.91 mm to (141.2, 102.3)
- moved J5 3.86 mm to (147.1, 92.0)
Routing:
- net Net-(J1-Pad3): track 117.9 -> 103.0 mm
- net Net-(J1-Pad1): track 120.5 -> 109.2 mm
- net Net-(J1-Pad2): track 128.2 -> 119.7 mm
Other:
- board text added: "D"
- board text added: "G"
- board text added: "Temperature HAT"
- board text removed: "Temperature HAT (based on DS18B20)"
