File: KiCad/pcb-hat-thermo/pcb-hat-thermo.kicad_sch (KiCad schematic)
At the start: 7 parts, among them J1 Screw_Terminal_01x03, J2 Screw_Terminal_01x03, J3 Screw_Terminal_01x03, J4 Screw_Terminal_01x03, J5 Screw_Terminal_01x03, J6 Raspberry_Pi_2_3

Commit message: Version 1.0
Parts:
- J1, J2, J3, J4, J5: footprint TerminalBlock_4Ucon:TerminalBlock_4Ucon_1x03_P3.50mm_Horizontal -> Connector_Phoenix_MC:PhoenixContact_MC_1,5_3-G-3.5_1x03_P3.50mm_Horizontal
- J6: footprint pcb-hat-lib:Raspberry_Pi_Zero_Custom -> pcb-hat-lib:Raspberry_Pi_Zero_Custom_with_Header
Changed lines of the file:
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@@
     (property "Reference" "J3" (id 0) (at 90.17 82.55 0))
     (property "Value" "Screw_Terminal_01x03" (id 1) (at 90.17 85.09 0))
-    (property "Footprint" "TerminalBlock_4Ucon:TerminalBlock_4Ucon_1x03_P3.50mm_Horizontal" (id 2) (at 90.17 91.44 0)
+    (property "Footprint" "Connector_Phoenix_MC:PhoenixContact_MC_1,5_3-G-3.5_1x03_P3.50mm_Horizontal" (id 2) (at 90.17 91.44 0)
       (effects (font (size 1.27 1.27)) hide)
     )
@@
     (property "Reference" "J4" (id 0) (at 90.17 97.79 0))
     (property "Value" "Screw_Terminal_01x03" (id 1) (at 90.17 100.33 0))
-    (property "Footprint" "TerminalBlock_4Ucon:TerminalBlock_4Ucon_1x03_P3.50mm_Horizontal" (id 2) (at 90.17 106.68 0)
+    (property "Footprint" "Connector_Phoenix_MC:PhoenixContact_MC_1,5_3-G-3.5_1x03_P3.50mm_Horizontal" (id 2) (at 90.17 106.68 0)
       (effects (font (size 1.27 1.27)) hide)
     )
@@
     (property "Reference" "J1" (id 0) (at 90.17 52.07 0))
     (property "Value" "Screw_Terminal_01x03" (id 1) (at 90.17 54.61 0))
-    (property "Footprint" "TerminalBlock_4Ucon:TerminalBlock_4Ucon_1x03_P3.50mm_Horizontal" (id 2) (at 90.17 60.96 0)
+    (property "Footprint" "Connector_Phoenix_MC:PhoenixContact_MC_1,5_3-G-3.5_1x03_P3.50mm_Horizontal" (id 2) (at 90.17 60.96 0)
       (effects (font (size 1.27 1.27)) hide)
     )
@@
       (effects (font (size 1.27 1.27)) (justify left))
     )
-    (property "Footprint" "pcb-hat-lib:Raspberry_Pi_Zero_Custom" (id 2) (at 168.91 87.63 0)
+    (property "Footprint" "pcb-hat-lib:Raspberry_Pi_Zero_Custom_with_Header" (id 2) (at 168.91 87.63 0)
       (effects (font (size 1.27 1.27)) hide)
     )
@@
     (property "Reference" "J2" (id 0) (at 90.17 67.31 0))
     (property "Value" "Screw_Terminal_01x03" (id 1) (at 90.17 69.85 0))
-    (property "Footprint" "TerminalBlock_4Ucon:TerminalBlock_4Ucon_1x03_P3.50mm_Horizontal" (id 2) (at 90.17 76.2 0)
+    (property "Footprint" "Connector_Phoenix_MC:PhoenixContact_MC_1,5_3-G-3.5_1x03_P3.50mm_Horizontal" (id 2) (at 90.17 76.2 0)
       (effects (font (size 1.27 1.27)) hide)
     )
@@
     (property "Reference" "J5" (id 0) (at 90.17 113.03 0))
     (property "Value" "Screw_Terminal_01x03" (id 1) (at 90.17 115.57 0))
-    (property "Footprint" "TerminalBlock_4Ucon:TerminalBlock_4Ucon_1x03_P3.50mm_Horizontal" (id 2) (at 90.17 121.92 0)
+    (property "Footprint" "Connector_Phoenix_MC:PhoenixContact_MC_1,5_3-G-3.5_1x03_P3.50mm_Horizontal" (id 2) (at 90.17 121.92 0)
       (effects (font (size 1.27 1.27)) hide)
     )
@@
     )
     (path "/72900501-da9e-4b56-869d-e5ada8646399"
-      (reference "J1") (unit 1) (value "Screw_Terminal_01x03") (footprint "TerminalBlock_4Ucon:TerminalBlock_4Ucon_1x03_P3.50mm_Horizontal")
+      (reference "J1") (unit 1) (value "Screw_Terminal_01x03") (footprint "Connector_Phoenix_MC:PhoenixContact_MC_1,5_3-G-3.5_1x03_P3.50mm_Horizontal")
     )
     (path "/8e2af090-a283-4b61-bfcb-a87fd64248fb"
-      (reference "J2") (unit 1) (value "Screw_Terminal_01x03") (footprint "TerminalBlock_4Ucon:TerminalBlock_4Ucon_1x03_P3.50mm_Horizontal")
+      (reference "J2") (unit 1) (value "Screw_Terminal_01x03") (footprint "Connector_Phoenix_MC:PhoenixContact_MC_1,5_3-G-3.5_1x03_P3.50mm_Horizontal")
     )
     (path "/28a418d9-a519-460d-a4e0-29c7ac183210"
-      (reference "J3") (unit 1) (value "Screw_Terminal_01x03") (footprint "TerminalBlock_4Ucon:TerminalBlock_4Ucon_1x03_P3.50mm_Horizontal")
+      (reference "J3") (unit 1) (value "Screw_Terminal_01x03") (footprint "Connector_Phoenix_MC:PhoenixContact_MC_1,5_3-G-3.5_1x03_P3.50mm_Horizontal")
     )
     (path "/30cd9c82-7ade-467e-870c-930f2e6dc805"
-      (reference "J4") (unit 1) (value "Screw_Terminal_01x03") (footprint "TerminalBlock_4Ucon:TerminalBlock_4Ucon_1x03_P3.50mm_Horizontal")
+      (reference "J4") (unit 1) (value "Screw_Terminal_01x03") (footprint "Connector_Phoenix_MC:PhoenixContact_MC_1,5_3-G-3.5_1x03_P3.50mm_Horizontal")
     )
     (path "/eb5c4588-833a-4b09-b41e-1f1f3533e07e"
-      (reference "J5") (unit 1) (value "Screw_Terminal_01x03") (footprint "TerminalBlock_4Ucon:TerminalBlock_4Ucon_1x03_P3.50mm_Horizontal")
+      (reference "J5") (unit 1) (value "Screw_Terminal_01x03") (footprint "Connector_Phoenix_MC:PhoenixContact_MC_1,5_3-G-3.5_1x03_P3.50mm_Horizontal")
     )
     (path "/896c762d-145f-49de-bc7f-0017853f4130"
-      (reference "J6") (unit 1) (value "Raspberry_Pi_2_3") (footprint "pcb-hat-lib:Raspberry_Pi_Zero_Custom")
+      (reference "J6") (unit 1) (value "Raspberry_Pi_2_3") (footprint "pcb-hat-lib:Raspberry_Pi_Zero_Custom_with_Header")
     )
     (path "/9f238e4c-0cbe-4d30-a10b-094d873a74e6"
